File: esp12-appliance-mod.kicad_pcb (KiCad board)
At the start: 2 copper layers, 76.2 x 76.2 mm, 41 parts, among them J1 CONN2, J2 CONN6, J3 CONN2, J4 CONN2, J5 CONN2, J6 CONN2, J7 CONN2, K1 RELAY_TE_RE314F05, Q1 MMBT4401, Q2 MMBT4401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

Commit message: Add part numbers to schematic. Regenerate BOM using BOMTools
Parts:
- J5: value CONN2 -> CONN2-3HSG
- J6, J7: value CONN2 -> CONN2-TB762
Connections:
- J2 pad 2: (no net) -> Net-(J2-Pad2)
- J2 pad 3: (no net) -> Net-(J2-Pad3)
- J2 pad 6: (no net) -> Net-(J2-Pad6)
- K1 pad 12A: (no net) -> Net-(K1-Pad12A)
- K1 pad 12B: (no net) -> Net-(K1-Pad12B)
- U1 pad 13: (no net) -> Net-(U1-Pad13)
- U1 pad 14: (no net) -> Net-(U1-Pad14)
- U1 pad 4: (no net) -> Net-(U1-Pad4)
